Commit message: moving my version of files into the branch

File: scripts/spherized.urdf (robot description, URDF)
Before this commit: robot panda, 13 links, 12 joints
Links:
- removed link panda_grasptarget
- removed link panda_hand
- removed link panda_leftfinger
- removed link panda_link0
- removed link panda_link1
- removed link panda_link2
- removed link panda_link3
- removed link panda_link4
- removed link panda_link5
- removed link panda_link6
- removed link panda_link7
- removed link panda_link8
- removed link panda_rightfinger
- added link base_link, mass 70.1294; collision sphere radius=0.358608; visual mesh filename=package://meshes/base_link.dae
- added link elbow_flex_link, mass 2.1299; collision sphere radius=0.073579; collision sphere radius=0.081094
- added link estop_link, mass 0.00196130439134723; visual mesh filename=package://meshes/estop_link.dae
- added link forearm_roll_link, mass 1.6563; collision sphere radius=0.060326; collision sphere radius=0.060464
- added link gripper_link, mass 1.5175; collision sphere radius=0.092125; visual mesh filename=package://meshes/gripper_link.dae
- added link head_camera_depth_frame
- added link head_camera_depth_optical_frame
- added link head_camera_link
- added link head_camera_rgb_frame
- added link head_camera_rgb_optical_frame
- added link head_pan_link, mass 2.2556; collision sphere radius=0.163316; collision sphere radius=0.176964
- added link head_tilt_link, mass 0.9087; collision sphere radius=0.089034; collision sphere radius=0.090387
- added link l_gripper_finger_link, mass 0.0798; collision sphere radius=0.0151; collision sphere radius=0.015493
- added link r_gripper_finger_link, mass 0.0798; collision sphere radius=0.015317; collision sphere radius=0.016059
- added link shoulder_lift_link, mass 2.6615; collision sphere radius=0.08775; collision sphere radius=0.095343
- added link shoulder_pan_link, mass 2.5587; collision sphere radius=0.096535; collision sphere radius=0.102167
- added link torso_fixed_link, mass 13.2775; collision sphere radius=0.191876; collision sphere radius=0.199625
- added link torso_lift_link, mass 10.7796; collision sphere radius=0.243207; collision sphere radius=0.254348
- added link upperarm_roll_link, mass 2.3311; collision sphere radius=0.063343; collision sphere radius=0.071761
- added link wrist_flex_link, mass 1.725; collision sphere radius=0.099854; visual mesh filename=package://meshes/wrist_flex_link.dae
- added link wrist_roll_link, mass 0.1354; collision sphere radius=0.056177; visual mesh filename=package://meshes/wrist_roll_link.dae
Joints:
- removed joint panda_finger_joint1
- removed joint panda_finger_joint2
- removed joint panda_grasptarget_hand
- removed joint panda_hand_joint
- removed joint panda_joint1
- removed joint panda_joint2
- removed joint panda_joint3
- removed joint panda_joint4
- removed joint panda_joint5
- removed joint panda_joint6
- removed joint panda_joint7
- removed joint panda_joint8
- added joint elbow_flex_joint: type revolute, parent upperarm_roll_link, child elbow_flex_link, origin xyz=0.133 0 0 rpy=0 0 0, axis 0 1 0, limit lower=-2.251 upper=2.251 effort=66.18 velocity=1.521
- added joint estop_joint: type fixed, parent base_link, child estop_link, origin xyz=-0.12465 0.23892 0.31127 rpy=1.5708 0 0, axis 0 0 0
- added joint forearm_roll_joint: type continuous, parent elbow_flex_link, child forearm_roll_link, origin xyz=0.197 0 0 rpy=0 0 0, axis 1 0 0, limit effort=29.35 velocity=1.571
- added joint gripper_axis: type fixed, parent wrist_roll_link, child gripper_link, origin xyz=0.16645 0 0 rpy=0 0 0, axis 0 1 0
- added joint head_camera_depth_joint: type fixed, parent head_camera_link, child head_camera_depth_frame, origin xyz=0 0.045 0 rpy=0 0 0
- added joint head_camera_depth_optical_joint: type fixed, parent head_camera_depth_frame, child head_camera_depth_optical_frame, origin xyz=0 0 0 rpy=-1.57079632679 0 -1.57079632679
- added joint head_camera_joint: type fixed, parent head_tilt_link, child head_camera_link, origin xyz=0.055 0 0.0225 rpy=0 0 0
- added joint head_camera_rgb_joint: type fixed, parent head_camera_link, child head_camera_rgb_frame, origin xyz=0 0.02 0 rpy=0 0 0
- added joint head_camera_rgb_optical_joint: type fixed, parent head_camera_rgb_frame, child head_camera_rgb_optical_frame, origin xyz=0 0 0 rpy=-1.57079632679 0 -1.57079632679
- added joint head_pan_joint: type fixed, parent torso_lift_link, child head_pan_link, origin xyz=0.053125 0 0.603001417713939 rpy=0 0 0, axis 0 0 1
- added joint head_tilt_joint: type fixed, parent head_pan_link, child head_tilt_link, origin xyz=0.14253 0 0.057999 rpy=0 0 0, axis 0 1 0
- added joint l_gripper_finger_joint: type fixed, parent gripper_link, child l_gripper_finger_link, origin xyz=0 -0.065425 0 rpy=0 0 0, axis 0 -1 0
- added joint r_gripper_finger_joint: type fixed, parent gripper_link, child r_gripper_finger_link, origin xyz=0 0.065425 0 rpy=0 0 0, axis 0 1 0
- added joint shoulder_lift_joint: type revolute, parent shoulder_pan_link, child shoulder_lift_link, origin xyz=0.117 0 0.0599999999999999 rpy=0 0 0, axis 0 1 0, limit lower=-1.221 upper=1.518 effort=131.76 velocity=1.454
- added joint shoulder_pan_joint: type revolute, parent torso_lift_link, child shoulder_pan_link, origin xyz=0.119525 0 0.34858 rpy=0 0 0, axis 0 0 1, limit lower=-1.6056 upper=1.6056 effort=33.82 velocity=1.256
- added joint torso_fixed_joint: type fixed, parent base_link, child torso_fixed_link, origin xyz=-0.086875 0 0.377425 rpy=-6.12303176911189E-17 0 0, axis 0 1 0
- added joint torso_lift_joint: type prismatic, parent base_link, child torso_lift_link, origin xyz=-0.086875 0 0.37743 rpy=-6.123E-17 0 0, axis 0 0 1, limit lower=0 upper=0.38615 effort=450.0 velocity=0.1
- added joint upperarm_roll_joint: type continuous, parent shoulder_lift_link, child upperarm_roll_link, origin xyz=0.219 0 0 rpy=0 0 0, axis 1 0 0, limit effort=76.94 velocity=1.571
- added joint wrist_flex_joint: type revolute, parent forearm_roll_link, child wrist_flex_link, origin xyz=0.1245 0 0 rpy=0 0 0, axis 0 1 0, limit lower=-2.16 upper=2.16 effort=25.7 velocity=2.268
- added joint wrist_roll_joint: type continuous, parent wrist_flex_link, child wrist_roll_link, origin xyz=0.1385 0 0 rpy=0 0 0, axis 1 0 0, limit effort=7.36 velocity=2.268
