Commit message: Worked on the preprocess test file. errors are present. Also corrected some minor issues in preprocess.py suych as the path to one of the assets.

File: spherized.urdf (robot description, URDF)
Before this commit: robot ur10e_robot, 11 links, 10 joints
Links:
- removed link base
- removed link base_link
- removed link base_link_inertia
- removed link flange
- removed link forearm_link
- removed link shoulder_link
- removed link tool0
- removed link upper_arm_link
- removed link wrist_1_link
- removed link wrist_2_link
- removed link wrist_3_link
- added link panda_grasptarget, mass 0.0
- added link panda_hand, mass .81; collision sphere radius=0.040412; collision sphere radius=0.044048
- added link panda_leftfinger, mass 0.1; collision sphere radius=0.015169; collision sphere radius=0.015906
- added link panda_link0, mass 2.9; collision sphere radius=0.092724; collision sphere radius=0.118826
- added link panda_link1, mass 2.7; collision sphere radius=0.088878; collision sphere radius=0.090742
- added link panda_link2, mass 2.73; collision sphere radius=0.077508; collision sphere radius=0.080094
- added link panda_link3, mass 2.04; collision sphere radius=0.082977; collision sphere radius=0.083241
- added link panda_link4, mass 2.08; collision sphere radius=0.081805; collision sphere radius=0.086213
- added link panda_link5, mass 3; collision sphere radius=0.070968; collision sphere radius=0.07761
- added link panda_link6, mass 1.3; collision sphere radius=0.074668; collision sphere radius=0.083093
- added link panda_link7, mass .2; collision sphere radius=0.049095; collision sphere radius=0.053568
- added link panda_link8, mass 0.0
- added link panda_rightfinger, mass 0.1; collision sphere radius=0.016951; collision sphere radius=0.017622
Joints:
- removed joint base_link-base_fixed_joint
- removed joint base_link-base_link_inertia
- removed joint elbow_joint
- removed joint flange-tool0
- removed joint shoulder_lift_joint
- removed joint shoulder_pan_joint
- removed joint wrist_1_joint
- removed joint wrist_2_joint
- removed joint wrist_3-flange
- removed joint wrist_3_joint
- added joint panda_finger_joint1: type fixed, parent panda_hand, child panda_leftfinger, origin xyz=0 0.065 0.0584 rpy=0 0 0, axis 0 1 0
- added joint panda_finger_joint2: type fixed, parent panda_hand, child panda_rightfinger, origin xyz=0 -0.065 0.0584 rpy=0 0 0, axis 0 -1 0, mimic joint=panda_finger_joint1
- added joint panda_grasptarget_hand: type fixed, parent panda_hand, child panda_grasptarget, origin xyz=0 0 0.105 rpy=0 0 0
- added joint panda_hand_joint: type fixed, parent panda_link8, child panda_hand, origin xyz=0 0 0 rpy=0 0 -0.785398163397
- added joint panda_joint1: type revolute, parent panda_link0, child panda_link1, origin xyz=0 0 0.333 rpy=0 0 0, axis 0 0 1, limit lower=-2.9671 upper=2.9671 effort=87 velocity=2.3925
- added joint panda_joint2: type revolute, parent panda_link1, child panda_link2, origin xyz=0 0 0 rpy=-1.57079632679 0 0, axis 0 0 1, limit lower=-1.8326 upper=1.8326 effort=87 velocity=2.3925
- added joint panda_joint3: type revolute, parent panda_link2, child panda_link3, origin xyz=0 -0.316 0 rpy=1.57079632679 0 0, axis 0 0 1, limit lower=-2.9671 upper=2.9671 effort=87 velocity=2.3925
- added joint panda_joint4: type revolute, parent panda_link3, child panda_link4, origin xyz=0.0825 0 0 rpy=1.57079632679 0 0, axis 0 0 1, limit lower=-3.1416 upper=0.0873 effort=87 velocity=2.3925
- added joint panda_joint5: type revolute, parent panda_link4, child panda_link5, origin xyz=-0.0825 0.384 0 rpy=-1.57079632679 0 0, axis 0 0 1, limit lower=-2.9671 upper=2.9671 effort=12 velocity=2.8710
- added joint panda_joint6: type revolute, parent panda_link5, child panda_link6, origin xyz=0 0 0 rpy=1.57079632679 0 0, axis 0 0 1, limit lower=-0.0873 upper=3.8223 effort=12 velocity=2.8710
- added joint panda_joint7: type revolute, parent panda_link6, child panda_link7, origin xyz=0.088 0 0 rpy=1.57079632679 0 0, axis 0 0 1, limit lower=-2.9671 upper=2.9671 effort=12 velocity=2.8710
- added joint panda_joint8: type fixed, parent panda_link7, child panda_link8, origin xyz=0 0 0.107 rpy=0 0 0, axis 0 0 0
